File: IEM_Crossover_Kicad/IEM_Crossover.kicad_pcb (KiCad board)
At the start: 2 copper layers, 5 parts, among them J1 0.78mm 2-pin

Commit message: Changed component footprints to 0805
Parts:
- R1, Z1, Z2: footprint Capacitor_SMD:C_01005_0402Metric -> Capacitor_SMD:C_0805_2012Metric
- moved J1 2.69 mm to (119.6, 83.6)
- moved D1 1.53 mm to (137.4, 82.2)
- moved Z1 0.44 mm to (125.9, 81.9)
