File: IEM_Crossover_Kicad/IEM_Crossover.kicad_sch (KiCad schematic)
At the start: 0 parts

Commit message: Added Branch 1, Created Driver Footprint
Parts:
- added D1: Speaker, Library:IEM_Driver_1x2_Pad, symbol Device:Speaker
- added J1: 0.78mm 2-pin, Library:IEM_Driver_1x2_Pad, symbol Connector:Conn_01x02_Pin
- added R1: R_Small, Capacitor_SMD:C_01005_0402Metric, symbol Device:R_Small
- added Z1, Z2: C_Small, Capacitor_SMD:C_01005_0402Metric, symbol Device:C_Small
Connections:
- new net: J1.1 (Pin_1), Z1.1
- new net: R1.1, Z1.2, Z2.2
- new net: D1.1, R1.2
- new net GND: D1.2, J1.2 (Pin_2), Z2.1

Commit message: Changed component footprints to 0805
Parts:
- R1, Z1, Z2: footprint Capacitor_SMD:C_01005_0402Metric -> Capacitor_SMD:C_0805_2012Metric
Changed lines of the file:
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@@
 			)
 		)
-		(property "Footprint" "Capacitor_SMD:C_01005_0402Metric"
+		(property "Footprint" "Capacitor_SMD:C_0805_2012Metric"
 			(at 91.44 77.47 0)
 			(hide yes)
@@
 		(in_pos_files yes)
 		(dnp no)
-		(fields_autoplaced yes)
 		(property "Reference" "R1"
-			(at 107.95 72.39 90)
+			(at 107.95 75.184 90)
 			(show_name no)
 			(do_not_autoplace no)
@@
 		(property "Value" "R_Small"
 			(at 107.95 74.93 90)
-			(show_name no)
-			(do_not_autoplace no)
-			(effects
-				(font
-					(size 1.27 1.27)
-				)
-			)
-		)
-		(property "Footprint" "Capacitor_SMD:C_01005_0402Metric"
+			(hide yes)
+			(show_name no)
+			(do_not_autoplace no)
+			(effects
+				(font
+					(size 1.27 1.27)
+				)
+			)
+		)
+		(property "Footprint" "Capacitor_SMD:C_0805_2012Metric"
 			(at 107.95 77.47 0)
 			(hide yes)
@@
 			)
 		)
-		(property "Footprint" "Capacitor_SMD:C_01005_0402Metric"
+		(property "Footprint" "Capacitor_SMD:C_0805_2012Metric"
 			(at 99.06 80.01 0)
 			(hide yes)
