File: IEM_Crossover_Kicad/IEM_Crossover.kicad_sch (KiCad schematic)
At the start: 5 parts, among them J1 0.78mm 2-pin

Commit message: finished layout
Parts:
- added B1, B2, C1, C2, D1, D2: C_Small, Capacitor_SMD:C_0805_2012Metric, symbol Device:C_Small
- added DR2, DR3, DR4: Speaker, Library:IEM_Driver_1x2_Pad, symbol Device:Speaker
- added R2, R3, R4: R_Small, Capacitor_SMD:C_0805_2012Metric, symbol Device:R_Small
- renumbered Z1 to A1, Z2 to A2, D1 to DR1
Connections:
- net GND: now also B2.1, C2.1, D2.1, DR2.2, DR3.2, DR4.2
- net at A1.1, J1.1 (Pin_1): now also B1.1, C1.1, D1.1
- new net: B1.2, B2.2, R2.1
- new net: DR2.1, R2.2
- new net: D1.2, D2.2, R4.1
- new net: C1.2, C2.2, R3.1
- new net: DR3.1, R3.2
- new net: DR4.1, R4.2
Other:
- moved on the sheet: A1, A2, DR1, R1
